Commit message: 增加ros插件

File: urdf/galileo_mini_x5.urdf (robot description, URDF)
Before this commit: robot galileo_mini_x5_description, 27 links, 26 joints
Links:
- link FL_abd_link: geometry collision cylinder length=0.1065 radius=0.06; visual mesh filename=package://galileo_mini_x5_description/meshes/FL_abd_link.STL
- link FL_hip_link: geometry collision box size=0.06 0.035 0.26; visual mesh filename=package://galileo_mini_x5_description/meshes/FL_hip_link.STL
- link FL_knee_link: geometry collision box size=0.05 0.03 0.23; visual mesh filename=package://galileo_mini_x5_description/meshes/FL_knee_link.S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
- link FR_abd_link: geometry collision cylinder length=0.1065 radius=0.06; visual mesh filename=package://galileo_mini_x5_description/meshes/FR_abd_link.STL
- link FR_hip_link: geometry collision box size=0.06 0.035 0.26; visual mesh filename=package://galileo_mini_x5_description/meshes/FR_hip_link.STL
- link FR_knee_link: geometry collision box size=0.05 0.03 0.23; visual mesh filename=package://galileo_mini_x5_description/meshes/FR_knee_link.S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
- link HL_abd_link: geometry collision cylinder length=0.1065 radius=0.06; visual mesh filename=package://galileo_mini_x5_description/meshes/HL_abd_link.STL
- link HL_hip_link: geometry collision box size=0.06 0.035 0.26; visual mesh filename=package://galileo_mini_x5_description/meshes/HL_hip_link.STL
- link HL_knee_link: geometry collision box size=0.05 0.03 0.23; visual mesh filename=package://galileo_mini_x5_description/meshes/HL_knee_link.S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
- link HR_abd_link: geometry collision cylinder length=0.1065 radius=0.06; visual mesh filename=package://galileo_mini_x5_description/meshes/HR_abd_link.STL
- link HR_hip_link: geometry collision box size=0.06 0.035 0.26; visual mesh filename=package://galileo_mini_x5_description/meshes/HR_hip_link.STL
- link HR_knee_link: geometry collision box size=0.05 0.03 0.23; visual mesh filename=package://galileo_mini_x5_description/meshes/HR_knee_link.S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
- link base_link: geometry collision box size=0.45 0.25 0.1; visual mesh filename=package://galileo_mini_x5_description/meshes/base_link.STL
- link link1: geometry visual mesh filename=package://galileo_mini_x5_description/meshes/link1.STL
- link link2: geometry visual mesh filename=package://galileo_mini_x5_description/meshes/link2.STL
- link link3: geometry visual mesh filename=package://galileo_mini_x5_description/meshes/link3.STL
- link link4: geometry visual mesh filename=package://galileo_mini_x5_description/meshes/link4.STL
- link link5: geometry visual mesh filename=package://galileo_mini_x5_description/meshes/link5.STL
- link link6: geometry visual mesh filename=package://galileo_mini_x5_description/meshes/link6.STL
- link link7: geometry visual mesh filename=package://galileo_mini_x5_description/meshes/link7.STL
- link link8: geometry visual mesh filename=package://galileo_mini_x5_description/meshes/link8.STL
- link manipulator_base_link: geometry visual mesh filename=package://galileo_mini_x5_description/meshes/manipulator_ba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
Joints:
- removed joint RR_foot_joint
- added joint HR_foot_joint: type fixed, parent HR_knee_link, child HR_foot_link, origin xyz=0.032939 0 -0.26149 rpy=0 0 0, axis 0 0 0
- joint FL_hip_joint: limit lower=-1.0472 upper=4.1888 effort=100 velocity=21 -> lower=-4.1888 upper=1.0472 effort=100 velocity=21
- joint FR_hip_joint: limit lower=-1.0472 upper=4.1888 effort=100 velocity=21 -> lower=-4.1888 upper=1.0472 effort=100 velocity=21
- joint HL_hip_joint: limit lower=-1.0472 upper=4.1888 effort=100 velocity=21 -> lower=-4.1888 upper=1.0472 effort=100 velocity=21
- joint HR_hip_joint: limit lower=-1.0472 upper=4.1888 effort=100 velocity=21 -> lower=-4.1888 upper=1.0472 effort=100 velocity=21
